File: pcb/_autosave-thermo.sch (KiCad schematic (older format))
At the start: 26 parts, among them J1 DB15_Female, J2 Barrel_Jack

Commit message: Add files via upload
Parts:
- 0.1uF1: renamed from 0.1uF; footprint (none) -> Capacitor_THT:C_Disc_D3.0mm_W1.6mm_P2.50mm
- ADC1, ADC2, ADC3, ADC4, ADC5: footprint (none) -> MAX31865:MAX31865
- ADC6, ADC7: footprint (none) -> MAX31856:MAX31856
- C1: renamed from C?; footprint (none) -> Capacitor_THT:CP_Radial_D5.0mm_P2.00mm
- MCU1: footprint (none) -> teensy:Teensy41
- Teensy_Ethernet1: renamed from Teensy_Ethernet; footprint (none) -> Connector_RJ:RJ45_Cetus_J1B1211CCD_Horizontal
- U1: renamed from U?; footprint (none) -> MAX31865:BME280
- gave numbers to parts that had none: 7
Changed lines of the file:
@@
 F 0 "MCU1" H 5700 6965 50  0000 C CNN
 F 1 "Teensy4.1" H 5700 6874 50  0000 C CNN
-F 2 "" H 5300 4800 50  0001 C CNN
+F 2 "teensy:Teensy41" H 5300 4800 50  0001 C CNN
 F 3 "" H 5300 4800 50  0001 C CNN
 	1    5700 4400
@@
 GND
 $Comp
-L Connector:RJ45_LED Teensy_Ethernet
+L Connector:RJ45_LED Teensy_Ethernet1
 U 1 1 612014A3
 P 8250 4950
-F 0 "Teensy_Ethernet" H 8250 5500 50  0000 C CNN
+F 0 "Teensy_Ethernet1" H 8250 5500 50  0000 C CNN
 F 1 "RJ45_LED" H 8100 4500 50  0000 C CNN
-F 2 "" V 8250 4975 50  0001 C CNN
+F 2 "Connector_RJ:RJ45_Cetus_J1B1211CCD_Horizontal" V 8250 4975 50  0001 C CNN
 F 3 "~" V 8250 4975 50  0001 C CNN
 	1    8250 4950
@@
 	6950 5000 6950 4750
 $Comp
-L power:GND #PWR?
+L power:GND #PWR0105
 U 1 1 6113FF3C
 P 7100 3750
-F 0 "#PWR?" H 7100 3500 50  0001 C CNN
+F 0 "#PWR0105" H 7100 3500 50  0001 C CNN
 F 1 "GND" H 7105 3577 50  0000 C CNN
 F 2 "" H 7100 3750 50  0001 C CNN
@@
 GND
 $Comp
-L Device:C 0.1uF
+L Device:C 0.1uF1
 U 1 1 6114C13E
 P 7400 5350
-F 0 "0.1uF" H 7515 5396 50  0000 L CNN
+F 0 "0.1uF1" H 7515 5396 50  0000 L CNN
 F 1 "C1" H 7515 5305 50  0000 L CNN
-F 2 "" H 7438 5200 50  0001 C CNN
-F 3 "~" H 7400 5350 50  0001 C CNN
+F 2 "Capacitor_THT:C_Disc_D3.0mm_W1.6mm_P2.50mm" H 7438 5200 50  0001 C CNN
+F 3 "Digikey BC1084CT-ND" H 7400 5350 50  0001 C CNN
 	1    7400 5350
 	1    0    0    -1
@@
 	7400 5200 7400 5250
 $Comp
-L Device:CP1 C?
+L Device:CP1 C1
 U 1 1 6115A1EB
 P 6450 1200
-F 0 "C?" H 6565 1246 50  0000 L CNN
+F 0 "C1" H 6565 1246 50  0000 L CNN
 F 1 "CP1" H 6565 1155 50  0000 L CNN
-F 2 "" H 6450 1200 50  0001 C CNN
+F 2 "Capacitor_THT:CP_Radial_D5.0mm_P2.00mm" H 6450 1200 50  0001 C CNN
 F 3 "~" H 6450 1200 50  0001 C CNN
 	1    6450 1200
@@
 F 0 "ADC1" H 2150 7050 50  0000 C CNN
 F 1 "PT100" H 2450 6050 50  0000 C CNN
-F 2 "" H 2300 6100 50  0001 C CNN
+F 2 "MAX31865:MAX31865" H 2300 6100 50  0001 C CNN
 F 3 "" H 2300 6100 50  0001 C CNN
 	1    2300 6550
@@
 F 0 "ADC2" H 2150 5950 50  0000 C CNN
 F 1 "PT100" H 2450 4950 50  0000 C CNN
-F 2 "" H 2300 5000 50  0001 C CNN
+F 2 "MAX31865:MAX31865" H 2300 5000 50  0001 C CNN
 F 3 "" H 2300 5000 50  0001 C CNN
 	1    2300 5450
@@
 F 0 "ADC3" H 2150 4850 50  0000 C CNN
 F 1 "PT100" H 2450 3850 50  0000 C CNN
-F 2 "" H 2300 3900 50  0001 C CNN
+F 2 "MAX31865:MAX31865" H 2300 3900 50  0001 C CNN
 F 3 "" H 2300 3900 50  0001 C CNN
 	1    2300 4350
@@
 F 0 "ADC4" H 2150 3750 50  0000 C CNN
 F 1 "PT100" H 2450 2750 50  0000 C CNN
-F 2 "" H 2300 2800 50  0001 C CNN
+F 2 "MAX31865:MAX31865" H 2300 2800 50  0001 C CNN
 F 3 "" H 2300 2800 50  0001 C CNN
 	1    2300 3250
@@
 F 0 "ADC7" V 4950 7350 50  0000 R CNN
 F 1 "thermocouple2" V 4950 6800 50  0000 R CNN
-F 2 "" H 5250 6450 50  0001 C CNN
+F 2 "MAX31856:MAX31856" H 5250 6450 50  0001 C CNN
 F 3 "" H 5250 6450 50  0001 C CNN
 	1    5250 6900
@@
 $EndComp
 $Comp
-L thermo_bme280:thermo_bme280 U?
+L thermo_bme280:thermo_bme280 U1
 U 1 1 611B16E5
 P 6400 6900
-F 0 "U?" V 6100 7300 50  0000 R CNN
+F 0 "U1" V 6100 7300 50  0000 R CNN
 F 1 "BME280" V 6100 6800 50  0000 R CNN
-F 2 "" H 6400 6450 50  0001 C CNN
+F 2 "MAX31865:BME280" H 6400 6450 50  0001 C CNN
 F 3 "" H 6400 6450 50  0001 C CNN
 	1    6400 6900
@@
 F 0 "ADC6" V 3750 7350 50  0000 R CNN
 F 1 "thermocouple1" V 3750 6800 50  0000 R CNN
-F 2 "" H 4050 6450 50  0001 C CNN
+F 2 "MAX31856:MAX31856" H 4050 6450 50  0001 C CNN
 F 3 "" H 4050 6450 50  0001 C CNN
 	1    4050 6900
@@
 F 0 "ADC5" H 2150 2650 50  0000 C CNN
 F 1 "PT100" H 2450 1650 50  0000 C CNN
-F 2 "" H 2300 1700 50  0001 C CNN
+F 2 "MAX31865:MAX31865" H 2300 1700 50  0001 C CNN
 F 3 "" H 2300 1700 50  0001 C CNN
 	1    2300 2150
@@
 	2650 1900 3100 1900
 $Comp
-L Device:R_Small_US R?
+L Device:R_Small_US R4
 U 1 1 611F5925
 P 2750 2100
-F 0 "R?" V 2700 2200 50  0000 C CNN
+F 0 "R4" V 2700 2200 50  0000 C CNN
 F 1 "22" V 2800 2200 50  0000 C CNN
 F 2 "" H 2750 2100 50  0001 C CNN
@@
 	0    1    1    0
 $EndComp
-Connection ~ 1950 4300
-Wire Wire Line
-	1950 4300 2150 4300
-Connection ~ 1950 4500
-Wire Wire Line
-	1950 4500 2150 4500
-Connection ~ 1950 4200
-Wire Wire Line
-	1950 4200 2150 4200
 Wire Wire Line
 	2650 4100 3100 4100
@@
 	2650 4700 3550 4700
 $Comp
-L Device:R_Small_US R?
+L Device:R_Small_US R5
 U 1 1 612429F9
 P 2750 4300
-F 0 "R?" V 2700 4400 50  0000 C CNN
+F 0 "R5" V 2700 4400 50  0000 C CNN
 F 1 "22" V 2800 4400 50  0000 C CNN
 F 2 "" H 2750 4300 50  0001 C CNN
@@
 	2650 5300 3100 5300
 $Comp
-L Device:R_Small_US R?
+L Device:R_Small_US R6
 U 1 1 6125C382
 P 2750 5400
-F 0 "R?" V 2700 5500 50  0000 C CNN
+F 0 "R6" V 2700 5500 50  0000 C CNN
 F 1 "22" V 2800 5500 50  0000 C CNN
 F 2 "" H 2750 5400 50  0001 C CNN
@@
 	2650 5800 3550 5800
 $Comp
-L Device:R_Small_US R?
+L Device:R_Small_US R7
 U 1 1 6128253D
 P 2750 6500
-F 0 "R?" V 2700 6600 50  0000 C CNN
+F 0 "R7" V 2700 6600 50  0000 C CNN
 F 1 "22" V 2800 6600 50  0000 C CNN
 F 2 "" H 2750 6500 50  0001 C CNN
@@
 	2650 6900 3550 6900
 $Comp
-L Device:R_Small_US R?
+L Device:R_Small_US R8
 U 1 1 612DA6D5
 P 4050 6450
-F 0 "R?" V 4000 6550 50  0000 C CNN
+F 0 "R8" V 4000 6550 50  0000 C CNN
 F 1 "22" V 4100 6550 50  0000 C CNN
 F 2 "" H 4050 6450 50  0001 C CNN
@@
 $EndComp
 $Comp
-L Device:R_Small_US R?
+L Device:R_Small_US R9
 U 1 1 612DB8DC
 P 5250 6450
-F 0 "R?" V 5200 6550 50  0000 C CNN
+F 0 "R9" V 5200 6550 50  0000 C CNN
 F 1 "22" V 5300 6550 50  0000 C CNN
 F 2 "" H 5250 6450 50  0001 C CNN
@@
 SDI
 $Comp
-L Device:R_Small_US R?
+L Device:R_Small_US R10
 U 1 1 612F54EE
 P 6300 6450
-F 0 "R?" V 6250 6550 50  0000 C CNN
+F 0 "R10" V 6250 6550 50  0000 C CNN
 F 1 "22" V 6350 6550 50  0000 C CNN
 F 2 "" H 6300 6450 50  0001 C CNN
@@
 Wire Wire Line
 	6300 6150 6300 6350
+Wire Wire Line
+	3550 2300 3550 2500
 Wire Wire Line
 	7550 2550 8150 2550
@@
 Wire Bus Line
 	3200 1650 3200 6050
-Wire Wire Line
-	3550 2300 3550 2500
 $EndSCHEMATC
