File: pcb/thermo.kicad_pcb (KiCad board)
At the start: 2 copper layers, 9 parts

Commit message: Pre-adding traces
Parts:
- removed ?: MAX31865, MAX31865:MAX31865
- removed REF**: DSUB-15_Female_Horizontal_P2.77x2.84mm_EdgePinOffset4.94mm_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, Connector_Dsub:DSUB-15_Female_Horizontal_P2.77x2.84mm_EdgePinOffset4.94mm_Housed_MountingHolesOffset7.48mm
- removed REF**: PinSocket_1x24_P2.54mm_Vertical, Connector_PinSocket_2.54mm:PinSocket_1x24_P2.54mm_Vertical
- removed REF**: BarrelJack_Horizontal, Connector_BarrelJack:BarrelJack_Horizontal
- removed REF**: RJ45_Cetus_J1B1211CCD_Horizontal, Connector_RJ:RJ45_Cetus_J1B1211CCD_Horizontal
- removed REF** (x2): MAX31856, MAX31856:MAX31856
- removed REF**: BME280, MAX31865:BME280
- removed REF**: Teensy 4.1, teensy:Teensy41
- added 0.1uF1: C1, Capacitor_THT:C_Disc_D3.0mm_W1.6mm_P2.50mm, F.Cu at (47.0, 83.8)
- added ADC1: PT100, Thermometry:MAX31865, F.Cu at (67.3, 76.2)
- added ADC2: PT100, Thermometry:MAX31865, F.Cu at (95.2, 76.2)
- added ADC3: PT100, Thermometry:MAX31865, F.Cu at (123.2, 76.2)
- added ADC4: PT100, Thermometry:MAX31865, F.Cu at (96.5, 139.7)
- added ADC5: PT100, Thermometry:MAX31865, F.Cu at (124.5, 139.7)
- added ADC6: thermocouple1, Thermometry:MAX31856, F.Cu at (158.8, 73.7)
- added ADC7: thermocouple2, Thermometry:MAX31856, F.Cu at (158.8, 142.2)
- added CP1: 47uF, Capacitor_THT:CP_Radial_D5.0mm_P2.00mm, F.Cu at (39.4, 133.3)
- added F1: 1A, Thermometry:thermo_fuse, F.Cu at (43.2, 124.5)
- added ILI9341TFT1: Conn_01x14, Thermometry:ILI9341_1x14_connector, F.Cu at (114.6, 109.7)
- added J1: DB15_Female, Thermometry:D15_Female_Horizontal, F.Cu at (161.3, 108.0)
- added J2: Barrel_Jack, Connector_BarrelJack:BarrelJack_Horizontal, F.Cu at (33.0, 125.7)
- added MCU1: Teensy4.1, Thermometry:Teensy41, F.Cu at (49.5, 108.0)
- added R1: 22, Resistor_SMD:R_0805_2012Metric_Pad1.20x1.40mm_HandSolder, F.Cu at (63.5, 123.2)
- added R10: 22, Resistor_SMD:R_0805_2012Metric_Pad1.20x1.40mm_HandSolder, F.Cu at (53.3, 121.9)
- added R2: 22, Resistor_SMD:R_0805_2012Metric_Pad1.20x1.40mm_HandSolder, F.Cu at (53.3, 95.2)
- added R3: 22, Resistor_SMD:R_0805_2012Metric_Pad1.20x1.40mm_HandSolder, F.Cu at (95.2, 121.9)
- added R4: 22, Resistor_SMD:R_0805_2012Metric_Pad1.20x1.40mm_HandSolder, F.Cu at (123.2, 120.7)
- added R5: 22, Resistor_SMD:R_0805_2012Metric_Pad1.20x1.40mm_HandSolder, F.Cu at (124.5, 95.2)
- added R6: 22, Resistor_SMD:R_0805_2012Metric_Pad1.20x1.40mm_HandSolder, F.Cu at (96.5, 95.2)
- added R7: 22, Resistor_SMD:R_0805_2012Metric_Pad1.20x1.40mm_HandSolder, F.Cu at (68.6, 95.2)
- added R8: 22, Resistor_SMD:R_0805_2012Metric_Pad1.20x1.40mm_HandSolder, F.Cu at (143.2, 73.7)
- added R9: 22, Resistor_SMD:R_0805_2012Metric_Pad1.20x1.40mm_HandSolder, F.Cu at (143.5, 142.2)
- added Teensy_Ethernet1: RJ45_LED, Connector_RJ:RJ45_Cetus_J1B1211CCD_Horizontal, F.Cu at (36.8, 81.3)
- added U1: BME280, Thermometry:BME280, F.Cu at (68.6, 134.6)
Routing:
- net /5V: track 0.00 -> 40.9 mm
- net GND: track 0.00 -> 34.1 mm
- net Net-(CP1-Pad1): track 0.00 -> 18.0 mm
Other:
- net class Default: clearance 0.2 -> 0.254; trace_width 0.25 -> 0.254; via_dia 0.8 -> 0.762; via_drill 0.4 -> 0.381
- rule pad_to_mask_clearance: 0 -> 0.000051
- rule trace_clearance: 0.2 -> 0.254

Commit message: Latest upload for Brian to check
Parts:
- added ILI9341TFT2: Conn_01x14, Thermometry:ILI9341_2x7_connector, F.Cu at (32.8, 79.0)
- added ILI9341TFT3: Conn_01x14, Thermometry:ILI9341_1x14_connector, F.Cu at (20.6, 79.2)
- added R11: 22, Resistor_SMD:R_0805_2012Metric_Pad1.20x1.40mm_HandSolder, F.Cu at (88.4, 116.3)
- ILI9341TFT1: footprint Thermometry:ILI9341_1x14_connector -> Thermometry:ILI9341_2x7_connector
- moved ADC7 49.2 mm to (134.6, 99.3)
- moved R9 48.8 mm to (120.4, 99.3), turned to 0 degrees
- moved Teensy_Ethernet1 41.4 mm to (35.1, 122.7)
- moved 0.1uF1 40.4 mm to (42.2, 124.0), turned to 90 degrees
- moved J1 34.1 mm to (137.4, 132.3)
- moved R8 31.0 mm to (119.4, 93.5), turned to 90 degrees
- moved ADC6 24.1 mm to (134.6, 73.9)
- moved ILI9341TFT1 21.2 mm to (93.5, 108.0)
- moved F1 18.6 mm to (41.4, 143.0)
- moved J2 17.1 mm to (31.2, 142.7)
- moved R5 13.3 mm to (111.3, 93.5)
- moved ADC3 13.2 mm to (110.0, 75.7)
- moved R6 11.8 mm to (84.8, 93.5)
- moved ADC2 11.7 mm to (83.6, 75.7)
- moved R7 10.6 mm to (58.2, 93.5)
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Connections:
- ILI9341TFT1 pad 9: /SDO -> Net-(ILI9341TFT1-Pad9)
- MCU1 pad 30: Net-(MCU1-Pad30) -> /CS_8
Routing:
- net +3V3: track 0.00 -> 468.3 mm, vias 0 -> 1
- net GND: track 34.1 -> 417.7 mm, vias 0 -> 1
- net /SDI: track 0.00 -> 306.6 mm, vias 0 -> 5
- net /CLK: track 0.00 -> 300.6 mm
- net /SDO: track 0.00 -> 220.3 mm
- net Net-(ADC1-Pad10): track 0.00 -> 183.5 mm
- net Net-(ADC1-Pad12): track 0.00 -> 164.4 mm
- net Net-(ADC1-Pad9): track 0.00 -> 163.7 mm
- net Net-(ADC3-Pad9): track 0.00 -> 111.9 mm
- net Net-(ADC3-Pad10): track 0.00 -> 93.4 mm
- net Net-(ADC3-Pad12): track 0.00 -> 84.5 mm
- net /CS_6: track 0.00 -> 70.2 mm, vias 0 -> 1
- net Net-(ADC4-Pad12): track 0.00 -> 57.8 mm
- net Net-(0.1uF1-Pad2): track 0.00 -> 52.4 mm, vias 0 -> 1
- net Net-(ADC4-Pad10): track 0.00 -> 47.3 mm
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
Commit message: Revised latest for Brian to check
Routing:
- net Net-(ADC1-Pad12): track 164.4 -> 169.6 mm
- net Net-(ADC1-Pad9): track 163.7 -> 160.9 mm
- net Net-(ADC1-Pad10): track 183.5 -> 181.6 mm

Commit message: BM routing attempt
Parts:
- moved ILI9341TFT3 122.2 mm to (134.6, 123.2)
- moved ILI9341TFT2 99.4 mm to (125.7, 114.3)
- moved ADC6 97.4 mm to (62.2, 139.1), turned to 180 degrees
- moved R5 77.6 mm to (34.3, 83.5), turned to 270 degrees
- moved ADC3 77.2 mm to (32.8, 77.7)
- moved R8 67.1 mm to (61.2, 127.0), turned to 0 degrees
- moved ADC4 64.1 mm to (112.5, 77.7), turned to 0 degrees
- moved ADC7 61.5 mm to (87.6, 139.1), turned to 180 degrees
- moved R9 49.8 mm to (86.6, 135.9)
- moved J1 49.7 mm to (132.1, 83.0)
- moved F1 47.8 mm to (42.6, 95.2), turned to 180 degrees
- moved U1 46.4 mm to (109.2, 137.2), turned to 270 degrees
- moved J2 44.6 mm to (32.2, 98.2)
- moved R3 43.6 mm to (114.3, 84.8)
- moved R10 42.0 mm to (98.1, 139.7), turned to 0 degrees
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Routing:
- net +3V3: track 468.3 -> 244.1 mm
- net Net-(ADC1-Pad10): track 181.6 -> 51.2 mm
- net Net-(ADC1-Pad12): track 169.6 -> 40.1 mm
- net GND: track 417.7 -> 308.3 mm, vias 1 -> 0
- net Net-(ADC1-Pad9): track 160.9 -> 51.9 mm
- net Net-(ADC2-Pad9): track 0.00 -> 83.1 mm
- net Net-(ADC2-Pad10): track 0.00 -> 76.1 mm
- net Net-(ADC2-Pad12): track 0.00 -> 71.3 mm
- net /CS_6: track 70.2 -> 0.00 mm, vias 1 -> 0
- net /SDO: track 220.3 -> 265.0 mm, vias 0 -> 8
- net (no net): track 0.00 -> 44.2 mm
- net /CS_1: track 35.7 -> 0.00 mm
- net Net-(ADC6-Pad5): track 36.9 -> 3.81 mm
- net /CLK: track 300.6 -> 268.6 mm, vias 0 -> 1
- net /SDI: track 306.6 -> 279.4 mm
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Other:
- board text added: "PC-246-112-05-C00 EXOThermometry"
