File: pcb/thermo.sch (KiCad schematic (older format))
At the start: 18 parts, among them J1 DB15_Female, J2 Barrel_Jack

Commit message: Add files via upload
Ready for review
Parts:
- added 0.1uF: CP1, symbol Device:CP1
- added Teensy_Ethernet: RJ45_LED, symbol Connector:RJ45_LED
Connections:
- net labels added: 5V
- net labels removed: 3V3_out, DRDY, FLT, RDY, T_CLK, T_CS, T_DIN, T_DO, T_IRQ, VIN_TFT
- wire segments 150 -> 168

Commit message: Add files via upload
Parts:
- removed 0.1uF: CP1, symbol Device:CP1
- removed MAX31856_1, MAX31856_2: Conn_01x09, symbol Connector_Generic:Conn_01x09
- removed MAX31865_1, MAX31865_2, MAX31865_3, MAX31865_4, MAX31865_5: Conn_01x08, symbol Connector_Generic:Conn_01x08
- removed Terminal1, Terminal2, Terminal3, Terminal4, Terminal5: Conn_01x04, symbol Connector_Generic:Conn_01x04
- removed tc_flat_connector1, tc_flat_connector2: Conn_01x02, symbol Connector_Generic:Conn_01x02
- added 0.1uF1: C1, symbol Device:C
- added ADC1, ADC2, ADC3, ADC4, ADC5: PT100, MAX31865:MAX31865, symbol thermo-rescue:MAX31865-max31865
- added ADC6: thermocouple1, MAX31856:MAX31856, symbol thermo_max31856:thermo_max31856
- added ADC7: thermocouple2, MAX31856:MAX31856, symbol thermo_max31856:thermo_max31856
- added C1: CP1, symbol Device:CP1
- added F1: 1A, symbol Device:Fuse_Small
- added R1, R10, R2, R3, R4, R5, R6, R7, R8, R9: 22, symbol Device:R_Small_US
- added U1: BME280, MAX31865:BME280, symbol thermo_bme280:thermo_bme280
- MCU1: footprint (none) -> teensy:Teensy41
- Teensy_Ethernet1: renamed from Teensy_Ethernet; footprint (none) -> Connector_RJ:RJ45_Cetus_J1B1211CCD_Horizontal
Connections:
- net labels added: CS_8, T_CS, T_IRQ
- wire segments 168 -> 193
Other:
- moved on the sheet: J1

Commit message: Pre-adding traces
Parts:
- added J?: Conn_02x07_Counter_Clockwise, symbol Connector_Generic:Conn_02x07_Counter_Clockwise
- 0.1uF1: footprint (none) -> Capacitor_THT:C_Disc_D3.0mm_W1.6mm_P2.50mm
- ADC1, ADC2, ADC3, ADC4, ADC5: footprint MAX31865:MAX31865 -> Thermometry:MAX31865
- ADC6, ADC7: footprint MAX31856:MAX31856 -> Thermometry:MAX31856
- CP1: renamed from C1; value CP1 -> 47uF; footprint (none) -> Capacitor_THT:CP_Radial_D5.0mm_P2.00mm
- F1: footprint (none) -> Thermometry:thermo_fuse
- ILI9341TFT1: footprint (none) -> Thermometry:ILI9341_1x14_connector
- J1: footprint (none) -> Thermometry:D15_Female_Horizontal
- J2: footprint (none) -> Connector_BarrelJack:BarrelJack_Horizontal
- MCU1: footprint teensy:Teensy41 -> Thermometry:Teensy41; symbol teensy:Teensy4.1 -> thermo-rescue:Teensy4.1-teensy
- R1, R10, R2, R3, R4, R5, R6, R7, R8, R9: footprint (none) -> Resistor_SMD:R_0805_2012Metric_Pad1.20x1.40mm_HandSolder
- U1: footprint MAX31865:BME280 -> Thermometry:BME280
Changed lines of the file:
@@
 $EndDescr
 $Comp
-L teensy:Teensy4.1 MCU1
+L thermo-rescue:Teensy4.1-teensy MCU1
 U 1 1 610D658F
 P 5700 4400
 F 0 "MCU1" H 5700 6965 50  0000 C CNN
 F 1 "Teensy4.1" H 5700 6874 50  0000 C CNN
-F 2 "teensy:Teensy41" H 5300 4800 50  0001 C CNN
+F 2 "Thermometry:Teensy41" H 5300 4800 50  0001 C CNN
 F 3 "" H 5300 4800 50  0001 C CNN
 	1    5700 4400
@@
 F 0 "J2" H 5507 1475 50  0000 C CNN
 F 1 "Barrel_Jack" H 5507 1384 50  0000 C CNN
-F 2 "" H 5500 1110 50  0001 C CNN
-F 3 "~" H 5500 1110 50  0001 C CNN
+F 2 "Connector_BarrelJack:BarrelJack_Horizontal" H 5500 1110 50  0001 C CNN
+F 3 "https://www.digikey.com/en/products/detail/cui-devices/PJ-002A/96962" H 5500 1110 50  0001 C CNN
 	1    5450 1150
 	1    0    0    -1
@@
 F 0 "J1" H 800 3350 50  0000 L CNN
 F 1 "DB15_Female" H 800 5150 50  0000 L CNN
-F 2 "" H 950 4250 50  0001 C CNN
+F 2 "Thermometry:D15_Female_Horizontal" H 950 4250 50  0001 C CNN
 F 3 " ~" H 950 4250 50  0001 C CNN
 	1    950  4250
@@
 F 0 "0.1uF1" H 7515 5396 50  0000 L CNN
 F 1 "C1" H 7515 5305 50  0000 L CNN
-F 2 "" H 7438 5200 50  0001 C CNN
-F 3 "~" H 7400 5350 50  0001 C CNN
+F 2 "Capacitor_THT:C_Disc_D3.0mm_W1.6mm_P2.50mm" H 7438 5200 50  0001 C CNN
+F 3 "Digikey BC1084CT-ND" H 7400 5350 50  0001 C CNN
 	1    7400 5350
 	1    0    0    -1
@@
 	7400 5200 7400 5250
 $Comp
-L Device:CP1 C1
+L Device:CP1 CP1
 U 1 1 6115A1EB
 P 6450 1200
-F 0 "C1" H 6565 1246 50  0000 L CNN
-F 1 "CP1" H 6565 1155 50  0000 L CNN
-F 2 "" H 6450 1200 50  0001 C CNN
-F 3 "~" H 6450 1200 50  0001 C CNN
+F 0 "CP1" H 6565 1246 50  0000 L CNN
+F 1 "47uF" H 6565 1155 50  0000 L CNN
+F 2 "Capacitor_THT:CP_Radial_D5.0mm_P2.00mm" H 6450 1200 50  0001 C CNN
+F 3 "2368-VHT47M25-ND" H 6450 1200 50  0001 C CNN
 	1    6450 1200
 	1    0    0    -1
@@
 Text Label 7750 1850 0    50   ~ 0
 VIN
-$Comp
-L Connector_Generic:Conn_01x14 ILI9341TFT1
-U 1 1 6110AE8C
-P 8350 2450
-F 0 "ILI9341TFT1" H 8500 3150 50  0000 C CNN
-F 1 "Conn_01x14" H 8500 1650 50  0000 C CNN
-F 2 "" H 8350 2450 50  0001 C CNN
-F 3 "~" H 8350 2450 50  0001 C CNN
-	1    8350 2450
-	1    0    0    -1
-$EndComp
 Wire Wire Line
 	2850 6500 3100 6500
@@
 F 0 "ADC1" H 2150 7050 50  0000 C CNN
 F 1 "PT100" H 2450 6050 50  0000 C CNN
-F 2 "MAX31865:MAX31865" H 2300 6100 50  0001 C CNN
+F 2 "Thermometry:MAX31865" H 2300 6100 50  0001 C CNN
 F 3 "" H 2300 6100 50  0001 C CNN
 	1    2300 6550
@@
 F 0 "ADC2" H 2150 5950 50  0000 C CNN
 F 1 "PT100" H 2450 4950 50  0000 C CNN
-F 2 "MAX31865:MAX31865" H 2300 5000 50  0001 C CNN
+F 2 "Thermometry:MAX31865" H 2300 5000 50  0001 C CNN
 F 3 "" H 2300 5000 50  0001 C CNN
 	1    2300 5450
@@
 F 0 "ADC3" H 2150 4850 50  0000 C CNN
 F 1 "PT100" H 2450 3850 50  0000 C CNN
-F 2 "MAX31865:MAX31865" H 2300 3900 50  0001 C CNN
+F 2 "Thermometry:MAX31865" H 2300 3900 50  0001 C CNN
 F 3 "" H 2300 3900 50  0001 C CNN
 	1    2300 4350
@@
 F 0 "ADC4" H 2150 3750 50  0000 C CNN
 F 1 "PT100" H 2450 2750 50  0000 C CNN
-F 2 "MAX31865:MAX31865" H 2300 2800 50  0001 C CNN
+F 2 "Thermometry:MAX31865" H 2300 2800 50  0001 C CNN
 F 3 "" H 2300 2800 50  0001 C CNN
 	1    2300 3250
@@
 F 0 "ADC7" V 4950 7350 50  0000 R CNN
 F 1 "thermocouple2" V 4950 6800 50  0000 R CNN
-F 2 "MAX31856:MAX31856" H 5250 6450 50  0001 C CNN
+F 2 "Thermometry:MAX31856" H 5250 6450 50  0001 C CNN
 F 3 "" H 5250 6450 50  0001 C CNN
 	1    5250 6900
@@
 F 0 "U1" V 6100 7300 50  0000 R CNN
 F 1 "BME280" V 6100 6800 50  0000 R CNN
-F 2 "MAX31865:BME280" H 6400 6450 50  0001 C CNN
+F 2 "Thermometry:BME280" H 6400 6450 50  0001 C CNN
 F 3 "" H 6400 6450 50  0001 C CNN
 	1    6400 6900
@@
 F 0 "ADC6" V 3750 7350 50  0000 R CNN
 F 1 "thermocouple1" V 3750 6800 50  0000 R CNN
-F 2 "MAX31856:MAX31856" H 4050 6450 50  0001 C CNN
+F 2 "Thermometry:MAX31856" H 4050 6450 50  0001 C CNN
 F 3 "" H 4050 6450 50  0001 C CNN
 	1    4050 6900
@@
 F 0 "F1" H 6800 865 50  0000 C CNN
 F 1 "1A" H 6800 956 50  0000 C CNN
-F 2 "" H 6800 1050 50  0001 C CNN
+F 2 "Thermometry:thermo_fuse" H 6800 1050 50  0001 C CNN
 F 3 "https://www.digikey.com/en/products/detail/littelfuse-inc/0154001-DRTL/2520456" H 6800 1050 50  0001 C CNN
 	1    6800 1050
@@
 F 0 "R1" V 4400 3550 50  0000 C CNN
 F 1 "22" V 4500 3550 50  0000 C CNN
-F 2 "" H 4450 3450 50  0001 C CNN
+F 2 "Resistor_SMD:R_0805_2012Metric_Pad1.20x1.40mm_HandSolder" H 4450 3450 50  0001 C CNN
 F 3 "~" H 4450 3450 50  0001 C CNN
 	1    4450 3450
@@
 F 0 "R2" V 6900 3450 50  0000 C CNN
 F 1 "22" V 7000 3450 50  0000 C CNN
-F 2 "" H 6950 3550 50  0001 C CNN
+F 2 "Resistor_SMD:R_0805_2012Metric_Pad1.20x1.40mm_HandSolder" H 6950 3550 50  0001 C CNN
 F 3 "~" H 6950 3550 50  0001 C CNN
 	1    6950 3550
@@
 F 0 "R3" V 2700 3300 50  0000 C CNN
 F 1 "22" V 2800 3300 50  0000 C CNN
-F 2 "" H 2750 3200 50  0001 C CNN
+F 2 "Resistor_SMD:R_0805_2012Metric_Pad1.20x1.40mm_HandSolder" H 2750 3200 50  0001 C CNN
 F 3 "~" H 2750 3200 50  0001 C CNN
 	1    2750 3200
@@
 F 0 "ADC5" H 2150 2650 50  0000 C CNN
 F 1 "PT100" H 2450 1650 50  0000 C CNN
-F 2 "MAX31865:MAX31865" H 2300 1700 50  0001 C CNN
+F 2 "Thermometry:MAX31865" H 2300 1700 50  0001 C CNN
 F 3 "" H 2300 1700 50  0001 C CNN
 	1    2300 2150
@@
 F 0 "R4" V 2700 2200 50  0000 C CNN
 F 1 "22" V 2800 2200 50  0000 C CNN
-F 2 "" H 2750 2100 50  0001 C CNN
+F 2 "Resistor_SMD:R_0805_2012Metric_Pad1.20x1.40mm_HandSolder" H 2750 2100 50  0001 C CNN
 F 3 "~" H 2750 2100 50  0001 C CNN
 	1    2750 2100
@@
 F 0 "R5" V 2700 4400 50  0000 C CNN
 F 1 "22" V 2800 4400 50  0000 C CNN
-F 2 "" H 2750 4300 50  0001 C CNN
+F 2 "Resistor_SMD:R_0805_2012Metric_Pad1.20x1.40mm_HandSolder" H 2750 4300 50  0001 C CNN
 F 3 "~" H 2750 4300 50  0001 C CNN
 	1    2750 4300
@@
 F 0 "R6" V 2700 5500 50  0000 C CNN
 F 1 "22" V 2800 5500 50  0000 C CNN
-F 2 "" H 2750 5400 50  0001 C CNN
+F 2 "Resistor_SMD:R_0805_2012Metric_Pad1.20x1.40mm_HandSolder" H 2750 5400 50  0001 C CNN
 F 3 "~" H 2750 5400 50  0001 C CNN
 	1    2750 5400
@@
 F 0 "R7" V 2700 6600 50  0000 C CNN
 F 1 "22" V 2800 6600 50  0000 C CNN
-F 2 "" H 2750 6500 50  0001 C CNN
+F 2 "Resistor_SMD:R_0805_2012Metric_Pad1.20x1.40mm_HandSolder" H 2750 6500 50  0001 C CNN
 F 3 "~" H 2750 6500 50  0001 C CNN
 	1    2750 6500
@@
 F 0 "R8" V 4000 6550 50  0000 C CNN
 F 1 "22" V 4100 6550 50  0000 C CNN
-F 2 "" H 4050 6450 50  0001 C CNN
+F 2 "Resistor_SMD:R_0805_2012Metric_Pad1.20x1.40mm_HandSolder" H 4050 6450 50  0001 C CNN
 F 3 "~" H 4050 6450 50  0001 C CNN
 	1    4050 6450
@@
 F 0 "R9" V 5200 6550 50  0000 C CNN
 F 1 "22" V 5300 6550 50  0000 C CNN
-F 2 "" H 5250 6450 50  0001 C CNN
+F 2 "Resistor_SMD:R_0805_2012Metric_Pad1.20x1.40mm_HandSolder" H 5250 6450 50  0001 C CNN
 F 3 "~" H 5250 6450 50  0001 C CNN
 	1    5250 6450
@@
 F 0 "R10" V 6250 6550 50  0000 C CNN
 F 1 "22" V 6350 6550 50  0000 C CNN
-F 2 "" H 6300 6450 50  0001 C CNN
+F 2 "Resistor_SMD:R_0805_2012Metric_Pad1.20x1.40mm_HandSolder" H 6300 6450 50  0001 C CNN
 F 3 "~" H 6300 6450 50  0001 C CNN
 	1    6300 6450
@@
 Wire Wire Line
 	3550 2300 3550 2500
+$Comp
+L Connector_Generic:Conn_01x14 ILI9341TFT1
+U 1 1 6110AE8C
+P 8350 2450
+F 0 "ILI9341TFT1" H 8500 3150 50  0000 C CNN
+F 1 "Conn_01x14" H 8500 1650 50  0000 C CNN
+F 2 "Thermometry:ILI9341_1x14_connector" H 8350 2450 50  0001 C CNN
+F 3 "~" H 8350 2450 50  0001 C CNN
+	1    8350 2450
+	1    0    0    -1
+$EndComp
+Wire Bus Line
+	3200 6050 6300 6050
 Wire Wire Line
 	7550 2550 8150 2550
 Wire Wire Line
 	7550 2150 8150 2150
+Wire Bus Line
+	7650 1650 7650 3050
 Wire Wire Line
 	7400 1950 8150 1950
+Wire Bus Line
+	7250 1650 7250 4650
+Wire Bus Line
+	4100 1650 4100 3450
 Wire Bus Line
 	3200 6050 3200 6700
 Wire Bus Line
-	7250 1650 7250 4650
-Wire Bus Line
-	7650 1650 7650 3050
-Wire Bus Line
-	4100 1650 4100 3450
-Wire Bus Line
-	3200 6050 6300 6050
-Wire Bus Line
 	3200 1650 3200 6050
+$Comp
+L Connector_Generic:Conn_02x07_Counter_Clockwise J?
+U 1 1 6124D54B
+P 9450 2500
+F 0 "J?" H 9500 3017 50  0000 C CNN
+F 1 "Conn_02x07_Counter_Clockwise" H 9500 2926 50  0000 C CNN
+F 2 "" H 9450 2500 50  0001 C CNN
+F 3 "~" H 9450 2500 50  0001 C CNN
+	1    9450 2500
+	1    0    0    -1
+$EndComp
 $EndSCHEMATC

Commit message: Latest upload for Brian to check
Parts:
- removed J?: Conn_02x07_Counter_Clockwise, symbol Connector_Generic:Conn_02x07_Counter_Clockwise
- added ILI9341TFT2: Conn_01x14, Thermometry:ILI9341_2x7_connector, symbol Connector_Generic:Conn_01x14
- added ILI9341TFT3: Conn_01x14, Thermometry:ILI9341_1x14_connector, symbol Connector_Generic:Conn_01x14
- added R11: 22, Resistor_SMD:R_0805_2012Metric_Pad1.20x1.40mm_HandSolder, symbol Device:R_Small_US
- ILI9341TFT1: footprint Thermometry:ILI9341_1x14_connector -> Thermometry:ILI9341_2x7_connector
Connections:
- net +3V3: now also ILI9341TFT2.1 (Pin_1), ILI9341TFT2.4 (Pin_4), ILI9341TFT2.8 (Pin_8), ILI9341TFT3.1 (Pin_1), ILI9341TFT3.4 (Pin_4), ILI9341TFT3.8 (Pin_8)
- net CLK: now also ILI9341TFT2.10 (Pin_10), ILI9341TFT2.7 (Pin_7), ILI9341TFT3.10 (Pin_10), ILI9341TFT3.7 (Pin_7)
- net CS_8: now also MCU1.30 (38_CS1_IN1)
- net GND: now also ILI9341TFT2.2 (Pin_2), ILI9341TFT3.2 (Pin_2)
- net SDI: now also ILI9341TFT2.12 (Pin_12), ILI9341TFT2.6 (Pin_6), ILI9341TFT3.12 (Pin_12), ILI9341TFT3.6 (Pin_6)
- net SDO: now also ILI9341TFT2.13 (Pin_13), ILI9341TFT2.9 (Pin_9), ILI9341TFT3.13 (Pin_13), ILI9341TFT3.9 (Pin_9), R11.2; no longer ILI9341TFT1.9 (Pin_9)
- net TFT_CS: now also ILI9341TFT2.3 (Pin_3), ILI9341TFT3.3 (Pin_3)
- net TFT_DC: now also ILI9341TFT2.5 (Pin_5), ILI9341TFT3.5 (Pin_5)
- net T_CS: now also ILI9341TFT2.11 (Pin_11), ILI9341TFT3.11 (Pin_11)
- net T_IRQ: now also ILI9341TFT2.14 (Pin_14), ILI9341TFT3.14 (Pin_14)
- new net: ILI9341TFT1.9 (Pin_9), R11.1
Changed lines of the file:
@@
 	8150 2450 7750 2450
-Wire Wire Line
-	8150 2650 7750 2650
 Wire Wire Line
 	6800 2250 7150 2250
@@
 F 0 "ILI9341TFT1" H 8500 3150 50  0000 C CNN
 F 1 "Conn_01x14" H 8500 1650 50  0000 C CNN
-F 2 "Thermometry:ILI9341_1x14_connector" H 8350 2450 50  0001 C CNN
+F 2 "Thermometry:ILI9341_2x7_connector" H 8350 2450 50  0001 C CNN
 F 3 "~" H 8350 2450 50  0001 C CNN
 	1    8350 2450
 	1    0    0    -1
 $EndComp
+$Comp
+L Connector_Generic:Conn_01x14 ILI9341TFT2
+U 1 1 611F021F
+P 9300 2450
+F 0 "ILI9341TFT2" H 9150 3150 50  0000 C CNN
+F 1 "Conn_01x14" H 9150 1650 50  0000 C CNN
+F 2 "Thermometry:ILI9341_2x7_connector" H 9300 2450 50  0001 C CNN
+F 3 "~" H 9300 2450 50  0001 C CNN
+	1    9300 2450
+	1    0    0    -1
+$EndComp
+$Comp
+L Connector_Generic:Conn_01x14 ILI9341TFT3
+U 1 1 611EC952
+P 9900 2450
+F 0 "ILI9341TFT3" H 10050 3150 50  0000 C CNN
+F 1 "Conn_01x14" H 10050 1650 50  0000 C CNN
+F 2 "Thermometry:ILI9341_1x14_connector" H 9900 2450 50  0001 C CNN
+F 3 "~" H 9900 2450 50  0001 C CNN
+	1    9900 2450
+	1    0    0    -1
+$EndComp
+Wire Wire Line
+	9100 1850 9700 1850
+Wire Wire Line
+	9100 1950 9700 1950
+Wire Wire Line
+	9700 2050 9100 2050
+Wire Wire Line
+	9100 2150 9700 2150
+Wire Wire Line
+	9700 2250 9100 2250
+Wire Wire Line
+	9100 2350 9700 2350
+Wire Wire Line
+	9700 2450 9100 2450
+Wire Wire Line
+	9100 2550 9700 2550
+Wire Wire Line
+	9700 2650 9100 2650
+Wire Wire Line
+	9100 2750 9700 2750
+Wire Wire Line
+	9700 2850 9100 2850
+Wire Wire Line
+	9100 2950 9700 2950
+Wire Wire Line
+	9700 3050 9100 3050
+Wire Wire Line
+	9100 3150 9700 3150
+Text Label 9450 1850 0    50   ~ 0
+VIN
+Text Label 9450 1950 0    50   ~ 0
+GND
+Text Label 9450 2050 0    50   ~ 0
+TFT_CS
+Text Label 9450 2150 0    50   ~ 0
+VIN
+Text Label 9450 2350 0    50   ~ 0
+SDI
+Text Label 9450 2250 0    50   ~ 0
+TFT_DC
+Text Label 9450 2450 0    50   ~ 0
+CLK
+Text Label 9450 2550 0    50   ~ 0
+VIN
+Text Label 9450 2650 0    50   ~ 0
+SDO
+Text Label 9450 2750 0    50   ~ 0
+CLK
+Text Label 9450 2850 0    50   ~ 0
+T_CS
+Text Label 9450 2950 0    50   ~ 0
+SDI
+Text Label 9450 3050 0    50   ~ 0
+SDO
+Text Label 9450 3150 0    50   ~ 0
+T_IRQ
+Entry Wire Line
+	7150 4050 7250 4150
+Wire Wire Line
+	6800 4050 7150 4050
+Wire Wire Line
+	7550 2550 8150 2550
+Wire Wire Line
+	7550 2150 8150 2150
+Wire Wire Line
+	7400 1950 8150 1950
 Wire Bus Line
-	3200 6050 6300 6050
-Wire Wire Line
-	7550 2550 8150 2550
-Wire Wire Line
-	7550 2150 8150 2150
-Wire Bus Line
-	7650 1650 7650 3050
-Wire Wire Line
-	7400 1950 8150 1950
+	3200 6050 3200 6700
 Wire Bus Line
 	7250 1650 7250 4650
 Wire Bus Line
+	7650 1650 7650 3050
+Wire Bus Line
 	4100 1650 4100 3450
 Wire Bus Line
-	3200 6050 3200 6700
+	3200 6050 6300 6050
 Wire Bus Line
 	3200 1650 3200 6050
-$Comp
-L Connector_Generic:Conn_02x07_Counter_Clockwise J?
-U 1 1 6124D54B
-P 9450 2500
-F 0 "J?" H 9500 3017 50  0000 C CNN
-F 1 "Conn_02x07_Counter_Clockwise" H 9500 2926 50  0000 C CNN
-F 2 "" H 9450 2500 50  0001 C CNN
-F 3 "~" H 9450 2500 50  0001 C CNN
-	1    9450 2500
-	1    0    0    -1
-$EndComp
+Text Label 6950 4050 0    50   ~ 0
+CS_8
+$Comp
+L Device:R_Small_US R11
+U 1 1 612455D8
+P 8050 2650
+F 0 "R11" V 8000 2750 50  0000 C CNN
+F 1 "22" V 8100 2750 50  0000 C CNN
+F 2 "Resistor_SMD:R_0805_2012Metric_Pad1.20x1.40mm_HandSolder" H 8050 2650 50  0001 C CNN
+F 3 "~" H 8050 2650 50  0001 C CNN
+	1    8050 2650
+	0    1    1    0
+$EndComp
+Wire Wire Line
+	7950 2650 7750 2650
 $EndSCHEMATC
